Commit message: changes

File: Section11_Build_the_Robot/bumperbot_ws/src/bumperbot_description/urdf/bumperbot.urdf.xacro (robot description, xacro)
@@ -150,4 +150,6 @@
     <axis xyz="0 0 0" />
   </joint>
+<!-- BEGIN: IMU BLOCK -->
+<!--
   <link name="imu_link">
     <inertial>
@@ -178,4 +180,53 @@
     <axis xyz="0 0 0" />
   </joint>
+ -->
+<!-- END: IMU BLOCK -->
+  <!-- RealSense D435i Mount Link -->
+  <link name="d435i_link">
+    <inertial>
+      <origin xyz="0 0 0" rpy="0 0 0"/>
+      <mass value="0.075"/>
+      <inertia ixx="1e-5" iyy="1e-5" izz="1e-5" ixy="0" ixz="0" iyz="0"/>
+    </inertial>
+    <visual>
+      <origin xyz="0 0 0" rpy="0 0 0"/>
+      <geometry>
+        <box size="0.09 0.02 0.02"/>
+      </geometry>
+      <material name="black"/>
+    </visual>
+    <collision>
+      <origin xyz="0 0 0" rpy="0 0 0"/>
+      <geometry>
+        <box size="0.09 0.02 0.02"/>
+      </geometry>
+    </collision>
+  </link>
+  <joint name="d435i_joint" type="fixed">
+    <origin xyz="0.08 0 0.07" rpy="0 0 0"/>
+    <parent link="base_link"/>
+    <child link="d435i_link"/>
+  </joint>
+  <!-- IMU Link -->
+  <link name="d435i_imu_link"/>
+  <joint name="d435i_imu_joint" type="fixed">
+    <origin xyz="0 0 0" rpy="0 0 0"/>
+    <parent link="d435i_link"/>
+    <child link="d435i_imu_link"/>
+  </joint>
+  <!-- Depth Optical Frame -->
+  <link name="d435i_depth_link"/>
+  <joint name="d435i_depth_joint" type="fixed">
+    <origin xyz="0 0 0" rpy="-1.5708 0 -1.5708"/>
+    <parent link="d435i_link"/>
+    <child link="d435i_depth_link"/>
+  </joint>
+  <!-- RGB Optical Frame -->
+  <link name="d435i_rgb_link"/>
+  <joint name="d435i_rgb_joint" type="fixed">
+    <origin xyz="0 0 0" rpy="-1.5708 0 -1.5708"/>
+    <parent link="d435i_link"/>
+    <child link="d435i_rgb_link"/>
+  </joint>
   <link name="laser_link">
     <inertial>
